File: KiCAD files/Bara Senzori/BaraSenzori.kicad_sch (KiCad schematic)
At the start: 50 parts, among them J1 FFC3B07-08-T, U17 CD74HC4067SM

Commit message: Added PCB design
Parts:
- R1, R10, R11, R12, R13, R14, R15, R16, R17, R18, R19, R2, R20, R21, R22, R23, R24, R25, R26, R27, R28, R29, R3, R30, R31, R32, R4, R5, R6, R7, R8, R9: footprint (none) -> Resistor_SMD:R_0805_2012Metric_Pad1.20x1.40mm_HandSolder
- U1, U10, U11, U12, U13, U14, U15, U16, U2, U3, U4, U5, U6, U7, U8, U9: footprint (none) -> SMD4:ITR8307
