File: KiCAD files/Line_RC.kicad_sch (KiCad schematic)
At the start: 58 parts, among them IC1 ESP32-WROVER-E-N4R8, IC2 CP2102N-A02-GQFN28R, IC3 BC847BDW1T1G, IC4 TLV75533PDBVR, IC5 TPS563240DDCR, J1 XT60PW-M, J2 XT60PW-M, J3 Conn_01x03_ESC, J4 FFC3B07-08-T, J8 Motor OUT, J9 Motor OUT

Commit message: Modified schematic
Connections:
- net +3.3V: now also J4.2; no longer J4.1
- net +BATT: now also U2.4 (VCC)
- net A1: now also U2.2 (FI); no longer U1.2 (FI)
- net A2: now also U2.1 (BI); no longer U2.2 (FI)
- net B1: now also U1.2 (FI); no longer U1.1 (BI)
- net B2: now also U1.1 (BI); no longer U2.1 (BI)
- net GND: now also J4.1; no longer J4.8
- net S0: now also J4.8; no longer J4.3
- net S1: now also J4.7; no longer J4.4
- net S2: now also J4.6; no longer J4.5
- net S3: now also J4.5; no longer J4.6
- net Z: now also J4.4; no longer J4.2
- net ~{E}: now also J4.3; no longer J4.7
Other:
- moved on the sheet: C10, C11, C12, C2, C21, C22, C23, C24, C3, C4, C5, C6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
