File: KiCAD files/Line-RC/files/Line_RC.kicad_pcb (KiCad board)
At the start: 4 copper layers, 63 parts, among them IC1 CP2102N-A02-GQFN28R, IC2 BC847BDW1T1G, IC3 TPS563240DDCR, IC4 ESP32-WROVER-E-N4R8, IC5 TLV75533PDBVR, J1 FFC3B07-08-T, J3 Motor OUT, J4 XT60PW-M, J5 XT60PW-M, J6 Conn_01x03_ESC, J7 Motor OUT

Commit message: Finished the PCB and generated Gerber files
Parts:
- removed J1: FFC3B07-08-T, FFC3B07-T:FFC3B0708T
- added IR: PinHeader_1x19_P2.54mm_Vertical, Connector_PinHeader_2.54mm:PinHeader_1x19_P2.54mm_Vertical, F.Cu at (129.5, 66.8)
- added MUX: SSOP-24_5.3x8.2mm_P0.65mm, Package_SO:SSOP-24_5.3x8.2mm_P0.65mm, F.Cu at (152.3, 75.5)
- moved J4 145.6 mm to (188.8, 82.4), turned to 0 degrees
- moved C7 70.1 mm to (126.2, 114.0), turned to 180 degrees
- moved JP4 69.4 mm to (129.3, 92.8), turned to 90 degrees
- moved TP3 68.7 mm to (126.3, 106.2), turned to -90 degrees
- moved IC4 66.0 mm to (185.9, 125.9), turned to 0 degrees
- moved C9 66.0 mm to (122.2, 116.2), turned to 180 degrees
- moved TP4 64.3 mm to (125.7, 116.6), turned to 180 degrees
- moved R13 64.0 mm to (126.2, 109.0), turned to 180 degrees
- moved R14 64.0 mm to (126.2, 111.0), turned to 0 degrees
- moved C14 64.0 mm to (125.8, 90.0), turned to 0 degrees
- moved L1 63.8 mm to (122.2, 109.5)
- moved J5 63.5 mm to (108.7, 82.4), turned to 0 degrees
- moved IC3 63.1 mm to (122.2, 113.3), turned to 180 degrees
- moved IC5 62.4 mm to (125.8, 92.9), turned to 180 degrees
- moved C4 62.0 mm to (122.2, 106.2)
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Connections:
- IC4 pad 33: ESC -> PWM
Routing:
- net GND: track 28.5 -> 330.1 mm, vias 6 -> 49
- net (no net): track 0.00 -> 205.9 mm
- net +3.3V: track 9.26 -> 208.2 mm, vias 2 -> 6
- net +BATT: track 0.00 -> 196.1 mm
- net PWM: track 0.00 -> 118.2 mm, vias 0 -> 1
- net B1: track 0.00 -> 106.1 mm, vias 0 -> 2
- net B2: track 0.00 -> 104.6 mm, vias 0 -> 2
- net +5V: track 0.00 -> 91.8 mm, vias 0 -> 2
- net ~{E}: track 0.00 -> 80.8 mm, vias 0 -> 3
- net Z: track 0.00 -> 79.8 mm, vias 0 -> 3
- net S1: track 0.00 -> 77.9 mm, vias 0 -> 3
- net S0: track 0.00 -> 77.1 mm, vias 0 -> 3
- net S3: track 0.00 -> 73.2 mm, vias 0 -> 3
- net S2: track 0.00 -> 72.1 mm, vias 0 -> 3
- net G: track 0.00 -> 68.7 mm, vias 0 -> 2
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- added copper zone on B.Cu, net GND
- added copper zone on F.Cu, net GND
- added copper zone on In1.Cu, net GND
Other:
- board outline added: 240 x 77.6 mm

Commit message: Added silkscreen and 3d models
Other:
- board text added: "+"
- board text added: "+3.3V"
- board text added: "+5V"
- board text added: "+5V Intern"
- board text added: "+Batt"
- board text added: "-"
- board text added: "Baterie"
- board text added: "ESC"
- board text added: "Feedback Buck"
- board text added: "GND"
- board text added: "IR"
- board text added: "Int/Ext"
- board text added: "LDO Enable"
- board text added: "PWM ESC"
- board text added: "S0"
- board text added: "S1"
- board text added: "S10"
- board text added: "S11"
- board text added: "S12"
- board text added: "S13"
- board text added: "S14"
- board text added: "S15"
- board text added: "S2"
- board text added: "S3"
- board text added: "S4"
- board text added: "S5"
- board text added: "S6"
- board text added: "S7"
- board text added: "S8"
- board text added: "S9"
- board text added: "Status"
- board text added: "Suport N20"
- board text added: "Suport tije"
- board text added: "Suspend"

Commit message: updated pcb dimensions
Parts:
- added TP10: RX, TestPoint:TestPoint_Pad_D2.0mm, F.Cu at (197.4, 123.2)
- added TP7: 5V rail, TestPoint:TestPoint_Pad_D2.0mm, F.Cu at (122.3, 89.6)
- added TP8: 5V rail, TestPoint:TestPoint_Pad_D2.0mm, F.Cu at (162.2, 139.8)
- added TP9: RX, TestPoint:TestPoint_Pad_D2.0mm, F.Cu at (197.4, 121.3)
Connections:
- Q1 pad : (no net) -> GND
Routing:
- net USB_D+: track 19.8 -> 28.8 mm, vias 4 -> 3
- net GND: track 330.1 -> 336.9 mm, vias 49 -> 52
- net TXD0: track 50.4 -> 55.6 mm
- net RXD0: track 49.3 -> 53.5 mm
- net +3.3V: track 208.2 -> 211.8 mm
- net VBUS: track 18.4 -> 22.0 mm
- net RTS: track 4.80 -> 7.97 mm
- net Net-(IC2-B1): track 5.61 -> 7.30 mm
- net USB_D-: track 17.1 -> 18.2 mm
- net EN: track 37.3 -> 38.3 mm
- net B1: track 106.1 -> 107.0 mm
- net B2: track 104.6 -> 105.5 mm
- net GPIO0: track 53.5 -> 53.7 mm, vias 3 -> 2
Other:
- board text added: "LDO En"
- board text added: "RX"
- board text added: "TX"
- board text added: "VBUS"
- board text removed: "LDO Enable"
