File: KiCAD files/Line-RC/files/Line_RC.kicad_sch (KiCad schematic)
At the start: 58 parts, among them IC1 ESP32-WROVER-E-N4R8, IC2 CP2102N-A02-GQFN28R, IC3 BC847BDW1T1G, IC4 TLV75533PDBVR, IC5 TPS563240DDCR, J1 XT60PW-M, J2 XT60PW-M, J3 Conn_01x03_ESC, J4 FFC3B07-08-T, J8 Motor OUT, J9 Motor OUT

Commit message: Issue found wit boot option
Parts:
- added D?: Inolux_IN-P55TATRGB, LED_SMD:LED_Inolux_IN-P55TATRGB_PLCC6_5.0x5.5mm_P1.8mm, symbol LED:Inolux_IN-P55TATRGB
- added TP6: 5V USB, symbol Connector:TestPoint
Connections:
- net +5V: now also TP6.1
- net DTR: no longer IC3.1 (E2), R9.1
- net EN: no longer IC3.3 (C1)
- net RTS: no longer IC3.4 (E1), R10.2
- net at R10.1: no longer IC3.2 (B2)
- net at R9.2: no longer IC3.5 (B1)
- net GPIO2: no longer names the net of IC3.6 (C2)
- no-connect marks 33 -> 35
Other:
- moved on the sheet: C4, C5, C6, IC1, J4, R11

Commit message: Started PCB layout and routing
Parts:
- added R10, R11, R9: 1k, Resistor_SMD:R_0805_2012Metric_Pad1.20x1.40mm_HandSolder, symbol Device:R
- C1: renamed from C2; footprint (none) -> Capacitor_SMD:C_0805_2012Metric_Pad1.18x1.45mm_HandSolder
- C10: renamed from C4; footprint (none) -> Capacitor_SMD:C_0805_2012Metric_Pad1.18x1.45mm_HandSolder
- C11: renamed from C21; footprint (none) -> Capacitor_SMD:C_0805_2012Metric_Pad1.18x1.45mm_HandSolder
- C12: renamed from C22; footprint (none) -> Capacitor_SMD:C_0805_2012Metric_Pad1.18x1.45mm_HandSolder
- C13: renamed from C8; footprint (none) -> Capacitor_SMD:C_0805_2012Metric_Pad1.18x1.45mm_HandSolder
- C14: renamed from C7; footprint (none) -> Capacitor_SMD:C_0805_2012Metric_Pad1.18x1.45mm_HandSolder
- C15: renamed from C23; footprint (none) -> Capacitor_SMD:C_0805_2012Metric_Pad1.18x1.45mm_HandSolder
- C16: renamed from C24; footprint (none) -> Capacitor_SMD:C_0805_2012Metric_Pad1.18x1.45mm_HandSolder
- C2: renamed from C3; footprint (none) -> Capacitor_SMD:C_0805_2012Metric_Pad1.18x1.45mm_HandSolder
- C3: renamed from C1; footprint (none) -> Capacitor_SMD:C_0805_2012Metric_Pad1.18x1.45mm_HandSolder
- C4: renamed from C11; footprint (none) -> Capacitor_SMD:C_0805_2012Metric_Pad1.18x1.45mm_HandSolder
- C5: renamed from C12; footprint (none) -> Capacitor_SMD:C_0805_2012Metric_Pad1.18x1.45mm_HandSolder
- C6: footprint (none) -> Capacitor_SMD:C_0805_2012Metric_Pad1.18x1.45mm_HandSolder
- C7: renamed from C9; footprint (none) -> Capacitor_SMD:C_0805_2012Metric_Pad1.18x1.45mm_HandSolder
- C8: renamed from C5; footprint (none) -> Capacitor_SMD:C_0805_2012Metric_Pad1.18x1.45mm_HandSolder
- C9: renamed from C10; footprint (none) -> Capacitor_SMD:C_0805_2012Metric_Pad1.18x1.45mm_HandSolder
- IC3: renamed from IC5; footprint SOT95P280X110-6N -> TPS563240:SOT95P280X110-6N
- IC5: renamed from IC4; footprint SOT95P280X145-5N -> TLV75533PDBVR:SOT95P280X145-5N
- J1: renamed from J4; footprint FFC3B0708T -> FFC3B07-T:FFC3B0708T
- J3: renamed from J8; footprint (none) -> Connector_PinHeader_2.54mm:PinHeader_1x02_P2.54mm_Vertical
- J6: renamed from J3; footprint (none) -> Connector_PinHeader_2.54mm:PinHeader_1x03_P2.54mm_Vertical
- J7: renamed from J9; footprint (none) -> Connector_PinHeader_2.54mm:PinHeader_1x02_P2.54mm_Vertical
- JP2: renamed from JP3; footprint (none) -> Jumper:SolderJumper-2_P1.3mm_Bridged_RoundedPad1.0x1.5mm
- JP3: renamed from JP6; footprint (none) -> Capacitor_SMD:C_0805_2012Metric_Pad1.18x1.45mm_HandSolder
- JP4: renamed from JP2; footprint (none) -> Jumper:SolderJumper-2_P1.3mm_Open_RoundedPad1.0x1.5mm
- JP5: footprint (none) -> Jumper:SolderJumper-2_P1.3mm_Open_RoundedPad1.0x1.5mm
- JP6: renamed from JP4; footprint (none) -> Jumper:SolderJumper-2_P1.3mm_Open_RoundedPad1.0x1.5mm
- L1: footprint (none) -> Inductor_SMD:L_Neosid_SMS-ME3015
- Q1: footprint (none) -> CX90M-16P:CX90M-16P_HIR
- R1: renamed from R5; footprint (none) -> Resistor_SMD:R_0805_2012Metric_Pad1.20x1.40mm_HandSolder
- R12: renamed from R11; footprint (none) -> Resistor_SMD:R_0805_2012Metric_Pad1.20x1.40mm_HandSolder
- R13: renamed from R4; footprint (none) -> Resistor_SMD:R_0805_2012Metric_Pad1.20x1.40mm_HandSolder
- R14: renamed from R3; footprint (none) -> Resistor_SMD:R_0805_2012Metric_Pad1.20x1.40mm_HandSolder
- R15: renamed from R12; footprint (none) -> Resistor_SMD:R_0805_2012Metric_Pad1.20x1.40mm_HandSolder
- R2: renamed from R6; footprint (none) -> Resistor_SMD:R_0805_2012Metric_Pad1.20x1.40mm_HandSolder
- R3: renamed from R1; footprint (none) -> Resistor_SMD:R_0805_2012Metric_Pad1.20x1.40mm_HandSolder
- R4: renamed from R2; footprint (none) -> Resistor_SMD:R_0805_2012Metric_Pad1.20x1.40mm_HandSolder
- R5: renamed from R7; footprint (none) -> Resistor_SMD:R_0805_2012Metric_Pad1.20x1.40mm_HandSolder
- R6: renamed from R8; footprint (none) -> Resistor_SMD:R_0805_2012Metric_Pad1.20x1.40mm_HandSolder
- R7: renamed from R10; value 10k (1%) -> 10k; footprint (none) -> Resistor_SMD:R_0805_2012Metric_Pad1.20x1.40mm_HandSolder
- R8: renamed from R9; value 10k (1%) -> 10k; footprint (none) -> Resistor_SMD:R_0805_2012Metric_Pad1.20x1.40mm_HandSolder
- SB1: renamed from JP1; footprint (none) -> Jumper:SolderJumper-2_P1.3mm_Open_RoundedPad1.0x1.5mm
- TP1: renamed from TP6; footprint (none) -> TestPoint:TestPoint_Pad_D2.0mm
- TP2: renamed from TP1; footprint (none) -> TestPoint:TestPoint_Pad_D2.0mm
- TP3, TP5: footprint (none) -> TestPoint:TestPoint_Pad_D2.0mm
- TP4: renamed from TP2; footprint (none) -> TestPoint:TestPoint_Pad_D2.0mm
- TP6: renamed from TP4; footprint (none) -> TestPoint:TestPoint_Pad_D2.0mm
- U1, U2: footprint (none) -> Package_SO:SSOP-8_3.9x5.05mm_P1.27mm
- gave numbers to parts that had none: 1
- renumbered D4 to D3, D3 to D4, IC2 to IC1, IC3 to IC2, IC1 to IC4, J1 to J4, J2 to J5
Connections:
- net A1: now also IC4.26 (IO4), U1.2 (FI); no longer U2.2 (FI)
- net A2: now also IC4.29 (IO5), U1.1 (BI); no longer U2.1 (BI)
- net B1: now also IC4.30 (IO18), U2.2 (FI); no longer U1.2 (FI)
- net B2: now also IC4.31 (IO19), U2.1 (BI); no longer U1.1 (BI)
- net DTR: now also IC2.1 (E2), R7.2
- net EN: now also C10.1, IC2.3 (C1), IC4.3 (EN), R12.1
- net GND: now also Q1. (MID), R10.2, R11.2, R9.2
- net GPIO0: now also IC2.6 (C2), IC4.25 (IO0)
- net PWM: now also IC4.33 (IO21)
- net RTS: now also IC2.4 (E1), R8.1
- net RXD0: now also IC4.35 (TXD0)
- net S0: now also IC4.10 (IO25)
- net S1: now also IC4.11 (IO26)
- net S2: now also IC4.12 (IO27)
- net S3: now also IC4.13 (IO14)
- net TXD0: now also IC4.34 (RXD0)
- net Z: now also IC4.8 (IO32)
- net ~{E}: now also IC4.16 (IO13)
- net at R7.1: now also IC2.5 (B1)
- net at D5.1 (KB): now also R11.1
- net at D5.2 (KR): now also R10.1
- net at D5.3 (KG): now also R9.1
- net G: now reaches D5.4 (AG)
- net G: now also IC4.37 (IO23)
- net R: now reaches D5.5 (AR)
- net R: now also IC4.36 (IO22)
- net B: now reaches D5.6 (AB)
- net B: now also IC4.24 (IO2)
- net at R8.2: now also IC2.2 (B2)
Other:
- moved on the sheet: C10, C6, C8, D5, IC2, IC4, J1, R12, R7, R8

Commit message: added 3D renderings and saved the final schematic
Parts:
- removed J1: FFC3B07-08-T, FFC3B07-T:FFC3B0708T, symbol FFC3B07-08-T:FFC3B07-08-T
- added IR: Conn_01x16_Pin, symbol Connector:Conn_01x16_Pin
- added MUX: CD74HC4067SM, Package_SO:SSOP-24_5.3x8.2mm_P0.65mm, symbol 74xx:CD74HC4067SM
- added TP10: TX, TestPoint:TestPoint_Pad_D2.0mm, symbol Connector:TestPoint
- added TP7: +3.3V rail, TestPoint:TestPoint_Pad_D2.0mm, symbol Connector:TestPoint
- added TP8: VBUS, TestPoint:TestPoint_Pad_D2.0mm, symbol Connector:TestPoint
- added TP9: RX, TestPoint:TestPoint_Pad_D2.0mm, symbol Connector:TestPoint
Connections:
- net +3.3V: now also MUX.24 (VCC), TP7.1
- net GND: now also MUX.12 (GND)
- net RXD0: now also TP9.1
- net S0: now also MUX.10 (S0)
- net S1: now also MUX.11 (S1)
- net S2: now also MUX.14 (S2)
- net S3: now also MUX.13 (S3)
- net TXD0: now also TP10.1
- net VBUS: now also TP8.1
- net Z: now also MUX.1 (COM)
- net ~{E}: now also MUX.15 (~{E})
- new net: IR.1 (Pin_1), MUX.9 (I0)
- new net: IR.10 (Pin_10), MUX.22 (I9)
- new net: IR.11 (Pin_11), MUX.21 (I10)
- new net: IR.12 (Pin_12), MUX.20 (I11)
- new net: IR.13 (Pin_13), MUX.19 (I12)
- new net: IR.14 (Pin_14), MUX.18 (I13)
- new net: IR.15 (Pin_15), MUX.17 (I14)
- new net: IR.16 (Pin_16), MUX.16 (I15)
- new net: IR.2 (Pin_2), MUX.8 (I1)
- new net: IR.3 (Pin_3), MUX.7 (I2)
- new net: IR.4 (Pin_4), MUX.6 (I3)
- new net: IR.5 (Pin_5), MUX.5 (I4)
- new net: IR.6 (Pin_6), MUX.4 (I5)
- new net: IR.7 (Pin_7), MUX.3 (I6)
- new net: IR.8 (Pin_8), MUX.2 (I7)
- new net: IR.9 (Pin_9), MUX.23 (I8)
Other:
- note added: "Electronica de control"
- note added: "MCU and MUX"
- company: (none) -> TechForge Performance Team
- title: (none) -> Miguel - Line RC
- moved on the sheet: C10, C6, C8, D5, IC4, R10, R11, R12, R9
